Commit message: module2 updated

File: simulation/humanoid.urdf (robot description, URDF)
Before this commit: robot simple_humanoid, 9 links, 8 joints
Links:
- added link left_hip_roll_link, mass 0.01
- added link left_shoulder_roll_link, mass 0.01
- added link right_hip_roll_link, mass 0.01
- added link right_shoulder_roll_link, mass 0.01
- link left_foot: mass 0.5 -> 1.0
- link left_shin: mass 2.0 -> 3.0; geometry collision cylinder length=0.4 radius=0.05; visual cylinder length=0.4 radius=0.05
- link left_thigh: mass 3.0 -> 4.0; geometry collision cylinder length=0.4 radius=0.06; visual cylinder length=0.4 radius=0.06
- link left_upper_arm: mass 1.0 -> 1.5; geometry collision cylinder length=0.3 radius=0.04; visual cylinder length=0.3 radius=0.04
- link right_foot: mass 0.5 -> 1.0
- link right_shin: mass 2.0 -> 3.0; geometry collision cylinder length=0.4 radius=0.05; visual cylinder length=0.4 radius=0.05
- link right_thigh: mass 3.0 -> 4.0; geometry collision cylinder length=0.4 radius=0.06; visual cylinder length=0.4 radius=0.06
- link right_upper_arm: mass 1.0 -> 1.5; geometry collision cylinder length=0.3 radius=0.04; visual cylinder length=0.3 radius=0.04
- link torso: mass 10.0 -> 15.0
Joints:
- removed joint left_ankle
- removed joint left_hip
- removed joint left_shoulder
- removed joint right_ankle
- removed joint right_hip
- removed joint right_shoulder
- added joint left_ankle_roll: type revolute, parent left_shin, child left_foot, origin xyz=0 0 -0.4 rpy=0 0 0, axis 1 0 0, limit lower=-0.3 upper=0.3 effort=80 velocity=10
- added joint left_hip_roll: type revolute, parent left_hip_roll_link, child left_thigh, origin xyz=0 0 0 rpy=0 0 0, axis 1 0 0, limit lower=-0.5 upper=1.0 effort=150 velocity=10
- added joint left_hip_yaw: type revolute, parent torso, child left_hip_roll_link, origin xyz=0 0.1 -0.25 rpy=0 0 0, axis 0 0 1, limit lower=-0.7 upper=0.7 effort=120 velocity=10
- added joint left_shoulder_pitch: type revolute, parent left_shoulder_roll_link, child left_upper_arm, origin xyz=0 0 0 rpy=0 0 0, axis 0 1 0, limit lower=-3.14 upper=3.14 effort=60 velocity=10
- added joint left_shoulder_roll: type revolute, parent torso, child left_shoulder_roll_link, origin xyz=0 0.15 0.15 rpy=0 0 0, axis 1 0 0, limit lower=-0.5 upper=1.0 effort=60 velocity=10
- added joint right_ankle_roll: type revolute, parent right_shin, child right_foot, origin xyz=0 0 -0.4 rpy=0 0 0, axis 1 0 0, limit lower=-0.3 upper=0.3 effort=80 velocity=10
- added joint right_hip_roll: type revolute, parent right_hip_roll_link, child right_thigh, origin xyz=0 0 0 rpy=0 0 0, axis 1 0 0, limit lower=-1.0 upper=0.5 effort=150 velocity=10
- added joint right_hip_yaw: type revolute, parent torso, child right_hip_roll_link, origin xyz=0 -0.1 -0.25 rpy=0 0 0, axis 0 0 1, limit lower=-0.7 upper=0.7 effort=120 velocity=10
- added joint right_shoulder_pitch: type revolute, parent right_shoulder_roll_link, child right_upper_arm, origin xyz=0 0 0 rpy=0 0 0, axis 0 1 0, limit lower=-3.14 upper=3.14 effort=60 velocity=10
- added joint right_shoulder_roll: type revolute, parent torso, child right_shoulder_roll_link, origin xyz=0 -0.15 0.15 rpy=0 0 0, axis 1 0 0, limit lower=-1.0 upper=0.5 effort=60 velocity=10
- joint left_knee: limit lower=0 upper=2.8 effort=100 velocity=10 -> lower=0 upper=2.5 effort=150 velocity=10
- joint right_knee: limit lower=0 upper=2.8 effort=100 velocity=10 -> lower=0 upper=2.5 effort=150 velocity=10
